Commit message: add ros2_control and gazebo plugin config

File: urdf/diffdrive_robot.urdf.xacro (robot description, xacro)
@@ -7,6 +7,6 @@
     <xacro:property name="wheel_radius" value="0.05"/>
     <xacro:property name="wheel_width" value="0.03"/>
-    <xacro:property name="wheel_separation" value="0.25"/>
-    <xacro:property name="wheel_offset_x" value="0.3"/>
+    <xacro:property name="wheel_separation" value="0.22"/>
+    <xacro:property name="wheel_offset_x" value="0.1"/>
     <xacro:property name="wheel_offset_z" value="-0.02"/>
     <!-- Base link -->
@@ -77,3 +77,23 @@
         <child link="caster_link"/>
     </joint>
+    <ros2_control name="DiffDriveSystem" type="system">
+        <hardware>
+            <plugin>gazebo_ros2_control/GazeboSystem</plugin>
+        </hardware>
+        <joint name="left_wheel_joint">
+            <command_interface name="velocity"/>
+            <state_interface name="velocity"/>
+            <state_interface name="position"/>
+        </joint>
+        <joint name="right_wheel_joint">
+            <command_interface name="velocity"/>
+            <state_interface name="velocity"/>
+            <state_interface name="position"/>
+        </joint>
+    </ros2_control>
+    <gazebo>
+        <plugin filename="libgazebo_ros2_control.so" name="gazebo_ros2_control">
+            <!-- <parameter>$(find diffdrive_robot)/config/diffdrive_controllers.yaml</parameter> -->
+        </plugin>
+    </gazebo>
 </robot>
